Commit message: Inline PI, otherwise xacro complains:  Property wasn't defined: u'pi'

File: cartographer_ros/urdf/robot.urdf.xacro (robot description, xacro)
@@ -39,5 +39,5 @@
         <link name="${prefix}_wheel">
             <visual>
-                <origin xyz="0 0 0" rpy="${pi/2} 0 0"/>
+              <origin xyz="0 0 0" rpy="${3.14159265359/2} 0 0"/>
                 <geometry>
                     <cylinder length="0.05" radius="${wheel_radius}"/>

File: cartographer_ros/urdf/sensors/astra.urdf.xacro (robot description, xacro)
@@ -14,5 +14,5 @@
     <link name="${prefix}_rgb_frame"/>
     <joint name="${prefix}_rgb_optical_joint" type="fixed">
-      <origin xyz="0 0 0" rpy="${-pi/2} 0 ${-pi/2}" />
+      <origin xyz="0 0 0" rpy="${-3.14159265359/2} 0 ${-3.14159265359/2}" />
       <parent link="${prefix}_rgb_frame" />
       <child link="${prefix}_rgb_optical_frame" />
@@ -53,5 +53,5 @@
     <link name="${prefix}_depth_frame"/>
     <joint name="${prefix}_depth_optical_joint" type="fixed">
-      <origin xyz="0 0 0" rpy="${-pi/2} 0 ${-pi/2}" />
+      <origin xyz="0 0 0" rpy="${-3.14159265359/2} 0 ${-3.14159265359/2}" />
       <parent link="${prefix}_depth_frame" />
       <child link="${prefix}_depth_optical_frame" />
